File: pcb/orb.brd (EAGLE design)
At the start: 30.5 x 41.9 mm, 6 parts

Commit message: changed name of component to reflect it's where the sensor goes
Parts:
- renumbered JP4 to MPU6050
Changed lines of the file:
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@@
 <element name="JP3" library="SparkFun-Connectors" package="1X04" value="" x="19.05" y="3.81" rot="R90"/>
 <element name="ULN1" library="SparkFun-PowerIC" package="DIL18" value="" x="12.7" y="13.97" rot="R270"/>
-<element name="JP4" library="SparkFun-Connectors" package="1X08" value="" x="3.81" y="36.83"/>
+<element name="MPU6050" library="SparkFun-Connectors" package="1X08" value="" x="3.81" y="36.83"/>
 </elements>
 <signals>
@@
 </polygon>
 <contactref element="JP1" pad="2"/>
-<contactref element="JP4" pad="2"/>
+<contactref element="MPU6050" pad="2"/>
 <contactref element="JP2" pad="1"/>
 </signal>
@@
 <signal name="A4" class="2">
 <contactref element="JP5" pad="11"/>
-<contactref element="JP4" pad="4"/>
+<contactref element="MPU6050" pad="4"/>
 <wire x1="24.13" y1="8.89" x2="21.59" y2="10.16" width="0.4064" layer="16"/>
 <wire x1="21.59" y1="10.16" x2="21.59" y2="12.7" width="0.4064" layer="16"/>
@@
 <signal name="A5" class="2">
 <contactref element="JP5" pad="12"/>
-<contactref element="JP4" pad="3"/>
+<contactref element="MPU6050" pad="3"/>
 <wire x1="22.86" y1="6.35" x2="24.13" y2="6.35" width="0.635" layer="1"/>
 <wire x1="21.59" y1="7.62" x2="22.86" y2="6.35" width="0.635" layer="1"/>
@@
 <signal name="3V3">
 <contactref element="JP1" pad="1"/>
-<contactref element="JP4" pad="1"/>
+<contactref element="MPU6050" pad="1"/>
 <wire x1="2.54" y1="34.29" x2="1.27" y2="34.29" width="0.3048" layer="1"/>
 <wire x1="3.81" y1="35.56" x2="2.54" y2="34.29" width="0.3048" layer="1"/>
@@
 <signal name="D2">
 <contactref element="JP1" pad="3"/>
-<contactref element="JP4" pad="8"/>
+<contactref element="MPU6050" pad="8"/>
 <wire x1="6.35" y1="29.21" x2="1.27" y2="29.21" width="0.3048" layer="1"/>
 <wire x1="10.16" y1="33.02" x2="6.35" y2="29.21" width="0.3048" layer="1"/>
